File: Amadioha.kicad_pcb (KiCad board)
At the start: 4 copper layers, 74 x 51.7 mm, 64 parts, among them IC1 ACS37800KMACTR-030B3-I2C, J1 691137710002, J2 SW_Debug, J3 691137710002, K1 G6DN-1A-SL_DC5, Q1 BSS138, Q2 BSS138, Q3 BSS138, SW1 PTS815, U1 STM32WB55CGU6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

Commit message: PCB validation and manufacturing
Parts:
- added C21: 0u1, Capacitor_SMD:C_0603_1608Metric_Pad1.08x0.95mm_HandSolder, B.Cu at (93.5, 69.0)
- added SW2: PTS815, PS815_SJK:PTS815SJK250SMTRLFS, B.Cu at (93.9, 63.8)
- moved J3 2.25 mm to (127.0, 64.1)
- moved J1 1.88 mm to (138.7, 64.1)
- moved K1 1.61 mm to (119.3, 64.7)
- moved F1 1.35 mm to (145.6, 73.0)
- moved C16 0.96 mm to (138.0, 98.9)
- moved C17 0.96 mm to (138.1, 103.8)
- moved D2 0.96 mm to (137.2, 106.5)
- moved G*** 0.96 mm to (141.6, 86.3)
- moved PS1 0.96 mm to (138.9, 73.2)
- moved R16 0.96 mm to (141.8, 107.0)
- moved U2 0.96 mm to (142.8, 101.5)
Connections:
- U1 pad 42: unconnected-(U1-PA15-Pad42) -> /Pair
Routing:
- net /Pair: track 0.00 -> 26.1 mm, vias 0 -> 2
- net +5V: track 62.6 -> 60.8 mm
- net /K1_C: track 15.3 -> 14.6 mm
- net GND: track 8.81 -> 9.11 mm, vias 70 -> 67
- net /AC_L: vias 0 -> 10
- added copper zone on B.Cu, net /AC_L
Other:
- board size 74 x 51.7 mm -> 74 x 49.9 mm
- board text added: "${TITLE} ${REVISION}"
- board text added: "Pair"
- board text added: "~{RST}"

Commit message: revision norm.
Changed lines of the file:
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@@
 		(title "Amadioha")
 		(date "2025-12-11")
-		(rev "1.0")
+		(rev "2025.1.0")
 		(company "GeneMaris Technologies")
 		(comment 1 "Wall embedded Smart Switch")
@@
 	)
 	(gr_text "${TITLE} ${REVISION}"
-		(at 139.5 87 270)
+		(at 139.5 90.25 270)
 		(layer "B.SilkS")
 		(effects
